File: BME280/BME280.kicad_pcb (KiCad board)
At the start: 2 copper layers, 12.7 x 10.2 mm, 3 parts, among them J1 Conn_01x04_Male, J2 Conn_01x04_Male, U1 BME280

Commit message: add the zip files
Other:
- board text added: "BME280 REV1"
Changed lines of the file:
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@@
   (general
     (thickness 1.6)
-    (drawings 12)
+    (drawings 13)
     (tracks 16)
     (zones 0)
@@
       (drillshape 0)
       (scaleselection 1)
-      (outputdirectory ""))
+      (outputdirectory "/Users/kevinlutzer/Projects/breakout-boards/gerbers/BME280-V1/"))
   )
   (net 0 "")
@@
       (effects (font (size 1 1) (thickness 0.15)) (justify mirror))
     )
-    (fp_text user %R (at 0 -3.81 270) (layer B.Fab)
-      (effects (font (size 1 1) (thickness 0.15)) (justify mirror))
-    )
     (fp_line (start -0.635 1.27) (end 1.27 1.27) (layer B.Fab) (width 0.1))
     (fp_line (start 1.27 1.27) (end 1.27 -8.89) (layer B.Fab) (width 0.1))
@@
     (fp_line (start 1.8 -9.4) (end 1.8 1.8) (layer B.CrtYd) (width 0.05))
     (fp_line (start 1.8 1.8) (end -1.8 1.8) (layer B.CrtYd) (width 0.05))
+    (fp_text user %R (at 0 -3.81 270) (layer B.Fab)
+      (effects (font (size 1 1) (thickness 0.15)) (justify mirror))
+    )
     (pad 4 thru_hole oval (at 0 -7.62 180) (size 1.7 1.7) (drill 1) (layers *.Cu *.Mask)
       (net 4 SCK))
@@
     )
     (fp_text value Conn_01x04_Male (at 0 -9.95) (layer B.Fab) hide
-      (effects (font (size 1 1) (thickness 0.15)) (justify mirror))
-    )
-    (fp_text user %R (at 0 -3.81 270) (layer B.Fab)
       (effects (font (size 1 1) (thickness 0.15)) (justify mirror))
     )
@@
     (fp_line (start 1.8 -9.4) (end 1.8 1.8) (layer B.CrtYd) (width 0.05))
     (fp_line (start 1.8 1.8) (end -1.8 1.8) (layer B.CrtYd) (width 0.05))
+    (fp_text user %R (at 0 -3.81 270) (layer B.Fab)
+      (effects (font (size 1 1) (thickness 0.15)) (justify mirror))
+    )
     (pad 4 thru_hole oval (at 0 -7.62 180) (size 1.7 1.7) (drill 1) (layers *.Cu *.Mask)
       (net 8 SDO))
@@
     (fp_text value BME280 (at 0.015 2.535 90) (layer F.Fab) hide
       (effects (font (size 1 1) (thickness 0.15)))
-    )
-    (fp_text user %R (at 0 0 270) (layer F.Fab)
-      (effects (font (size 0.5 0.5) (thickness 0.075)))
     )
     (fp_line (start -1.35 1.36) (end -1.2 1.36) (layer F.SilkS) (width 0.1))
@@
     (fp_line (start 1.41 -1.54) (end 1.41 1.54) (layer F.CrtYd) (width 0.05))
     (fp_line (start 1.41 1.54) (end -1.41 1.54) (layer F.CrtYd) (width 0.05))
+    (fp_text user %R (at 0 0 270) (layer F.Fab)
+      (effects (font (size 0.5 0.5) (thickness 0.075)))
+    )
     (pad 5 smd rect (at 0.975 1.025) (size 0.5 0.35) (layers F.Cu F.Paste F.Mask)
       (net 8 SDO))
@@
     )
   )
+  (gr_text "BME280\nREV1" (at 185.547 106.426) (layer B.SilkS)
+    (effects (font (size 1 1) (thickness 0.15)) (justify mirror))
+  )
   (gr_text SDI (at 188.595 110.617) (layer F.SilkS)
