File: TSL25911FN/TSL25911FN.kicad_pcb (KiCad board)
At the start: 2 copper layers, 12.7 x 7.6 mm, 3 parts, among them J1 Conn_01x03_Male, J2 Conn_01x03_Male, U1 TSL2591

Commit message: add the zip files
Other:
- board text added: "TSL25911FN REV 1"
- board text removed: "TSL25911FN REV A"
Changed lines of the file:
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@@
   (general
     (thickness 1.6)
-    (drawings 11)
+    (drawings 13)
     (tracks 10)
     (zones 0)
@@
       (drillshape 0)
       (scaleselection 1)
-      (outputdirectory "/Users/kevinlutzer/Projects/breakout-boards/gerbers/TSL25911FN/"))
+      (outputdirectory "/Users/kevinlutzer/Projects/breakout-boards/gerbers/TSL25911FN-V1/"))
   )
   (net 0 "")
@@
       (effects (font (size 1 1) (thickness 0.15)))
     )
+    (fp_line (start -1.5 -1.5) (end 1.5 -1.5) (layer F.CrtYd) (width 0.06))
+    (fp_line (start -1.5 1.5) (end -1.5 -1.5) (layer F.CrtYd) (width 0.06))
+    (fp_line (start 1.5 1.5) (end -1.5 1.5) (layer F.CrtYd) (width 0.06))
+    (fp_line (start 1.5 -1.5) (end 1.5 1.5) (layer F.CrtYd) (width 0.06))
+    (fp_line (start 1 1.3) (end 0 1.3) (layer F.SilkS) (width 0.12))
+    (fp_line (start 1 -1.3) (end -1 -1.3) (layer F.SilkS) (width 0.12))
+    (fp_line (start 1 1.2) (end 1 1) (layer F.Fab) (width 0.12))
+    (fp_line (start -1 1.2) (end 1 1.2) (layer F.Fab) (width 0.12))
+    (fp_line (start -1 1) (end -1 1.2) (layer F.Fab) (width 0.12))
+    (fp_line (start -1 -1) (end -1 1) (layer F.Fab) (width 0.12))
+    (fp_line (start -1 -1.2) (end -1 -1) (layer F.Fab) (width 0.12))
+    (fp_line (start 1 -1.2) (end -1 -1.2) (layer F.Fab) (width 0.12))
+    (fp_line (start 1 -1) (end 1 -1.2) (layer F.Fab) (width 0.12))
+    (fp_line (start -1 -1.2) (end 0 -1.2) (layer F.Fab) (width 0.12))
+    (fp_line (start -1 1) (end -1 -1) (layer F.Fab) (width 0.12))
+    (fp_line (start 1 1.2) (end -1 1.2) (layer F.Fab) (width 0.12))
+    (fp_line (start 1 -1) (end 1 1) (layer F.Fab) (width 0.12))
     (fp_line (start 0 -1.2) (end 1 -1.2) (layer F.Fab) (width 0.12))
-    (fp_line (start 1 -1) (end 1 1) (layer F.Fab) (width 0.12))
-    (fp_line (start 1 1.2) (end -1 1.2) (layer F.Fab) (width 0.12))
-    (fp_line (start -1 1) (end -1 -1) (layer F.Fab) (width 0.12))
-    (fp_line (start -1 -1.2) (end 0 -1.2) (layer F.Fab) (width 0.12))
-    (fp_line (start 1 -1) (end 1 -1.2) (layer F.Fab) (width 0.12))
-    (fp_line (start 1 -1.2) (end -1 -1.2) (layer F.Fab) (width 0.12))
-    (fp_line (start -1 -1.2) (end -1 -1) (layer F.Fab) (width 0.12))
-    (fp_line (start -1 -1) (end -1 1) (layer F.Fab) (width 0.12))
-    (fp_line (start -1 1) (end -1 1.2) (layer F.Fab) (width 0.12))
-    (fp_line (start -1 1.2) (end 1 1.2) (layer F.Fab) (width 0.12))
-    (fp_line (start 1 1.2) (end 1 1) (layer F.Fab) (width 0.12))
-    (fp_line (start 1 -1.3) (end -1 -1.3) (layer F.SilkS) (width 0.12))
-    (fp_line (start 1 1.3) (end 0 1.3) (layer F.SilkS) (width 0.12))
-    (fp_line (start 1.5 -1.5) (end 1.5 1.5) (layer F.CrtYd) (width 0.06))
-    (fp_line (start 1.5 1.5) (end -1.5 1.5) (layer F.CrtYd) (width 0.06))
-    (fp_line (start -1.5 1.5) (end -1.5 -1.5) (layer F.CrtYd) (width 0.06))
-    (fp_line (start -1.5 -1.5) (end 1.5 -1.5) (layer F.CrtYd) (width 0.06))
-    (pad 6 smd rect (at 0.75 -0.65) (size 1.2 0.35) (layers F.Cu)
+    (pad 6 smd rect (at 0.75 -0.65) (size 1.2 0.35) (layers F.Cu F.Paste F.Mask)
       (net 1 SDA))
-    (pad 5 smd rect (at 0.75 0) (size 1.2 0.35) (layers F.Cu)
+    (pad 5 smd rect (at 0.75 0) (size 1.2 0.35) (layers F.Cu F.Paste F.Mask)
       (net 2 VDD))
-    (pad 4 smd rect (at 0.75 0.65) (size 1.2 0.35) (layers F.Cu)
+    (pad 4 smd rect (at 0.75 0.65) (size 1.2 0.35) (layers F.Cu F.Paste F.Mask)
       (net 6 NC))
-    (pad 3 smd rect (at -0.75 0.65) (size 1.2 0.35) (layers F.Cu)
+    (pad 3 smd rect (at -0.75 0.65) (size 1.2 0.35) (layers F.Cu F.Paste F.Mask)
       (net 3 GND))
-    (pad 2 smd rect (at -0.75 0) (size 1.2 0.35) (layers F.Cu)
+    (pad 2 smd rect (at -0.75 0) (size 1.2 0.35) (layers F.Cu F.Paste F.Mask)
       (net 4 INT))
-    (pad 1 smd oval (at -0.75 -0.65) (size 1.2 0.35) (layers F.Cu)
+    (pad 1 smd oval (at -0.75 -0.65) (size 1.2 0.35) (layers F.Cu F.Paste F.Mask)
       (net 5 SCL))
   )
@@
     )
   )
-  (gr_text "TSL25911FN\nREV A" (at 149.86 74.422) (layer B.SilkS)
+  (dimension 12.7 (width 0.15) (layer Cmts.User)
+    (gr_text "12.700 mm" (at 149.86 83.469) (layer Cmts.User)
+      (effects (font (size 1 1) (thickness 0.15)))
+    )
+    (feature1 (pts (xy 156.21 80.01) (xy 156.21 82.755421)))
+    (feature2 (pts (xy 143.51 80.01) (xy 143.51 82.755421)))
+    (crossbar (pts (xy 143.51 82.169) (xy 156.21 82.169)))
+    (arrow1a (pts (xy 156.21 82.169) (xy 155.083496 82.755421)))
+    (arrow1b (pts (xy 156.21 82.169) (xy 155.083496 81.582579)))
+    (arrow2a (pts (xy 143.51 82.169) (xy 144.636504 82.755421)))
+    (arrow2b (pts (xy 143.51 82.169) (xy 144.636504 81.582579)))
+  )
+  (dimension 7.62 (width 0.15) (layer Cmts.User)
+    (gr_text "7.620 mm" (at 139.67 76.2 270) (layer Cmts.User)
+      (effects (font (size 1 1) (thickness 0.15)))
+    )
+    (feature1 (pts (xy 143.51 80.01) (xy 140.383579 80.01)))
+    (feature2 (pts (xy 143.51 72.39) (xy 140.383579 72.39)))
+    (crossbar (pts (xy 140.97 72.39) (xy 140.97 80.01)))
+    (arrow1a (pts (xy 140.97 80.01) (xy 140.383579 78.883496)))
+    (arrow1b (pts (xy 140.97 80.01) (xy 141.556421 78.883496)))
+    (arrow2a (pts (xy 140.97 72.39) (xy 140.383579 73.516504)))
+    (arrow2b (pts (xy 140.97 72.39) (xy 141.556421 73.516504)))
+  )
+  (gr_text NC (at 152.654 78.74) (layer F.SilkS)
+    (effects (font (size 1 1) (thickness 0.15)))
+  )
+  (gr_text "TSL25911FN\nREV 1" (at 149.86 74.422) (layer B.SilkS)
     (effects (font (size 0.9 0.9) (thickness 0.12)) (justify mirror))
   )
-  (gr_text NC (at 152.781 78.74) (layer F.SilkS)
-    (effects (font (size 0.8 0.8) (thickness 0.12)))
-  )
   (gr_text SDA (at 152.146 73.66) (layer F.SilkS)
