File: STM32F411CE/STM32F411CE/STM32F411CE.kicad_pcb (KiCad board)
At the start: 2 copper layers, 27.9 x 41.9 mm, 28 parts, among them J1 USB_B_Mini, J2 Conn_ARM_JTAG_SWD_10, J3 Conn_01x14_Male, J4 Connector_PinHeader_2.54mm:Pi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, SW1 SW_SPDT, SW2 SW_SPST, SW3 SW_SPST, U1 W25Q32JVSS, U2 USBLC6-2SC6, U3 STM32F411CEUx, Y1 Crystal_GND24

Commit message: WIP
Parts:
- removed C6: 0.1uF, Capacitor_SMD:C_0402_1005Metric_Pad0.74x0.62mm_HandSolder
- removed FB1: 10uH, Inductor_SMD:L_0603_1608Metric
- removed J4: Connector_PinHeader_2.54mm:PinHeader_1x14_P2.54mm_Vertical, Connector_PinHeader_2.54mm:PinHeader_1x14_P2.54mm_Vertical
- removed R1, R2, R3, R4, R5, R6: 10k, Resistor_SMD:R_0402_1005Metric
- removed SW1: SW_SPDT, Button_Switch_SMD:SW_SPDT_PCM12
- removed SW2, SW3: SW_SPST, Button_Switch_SMD:SW_Push_1P1T_NO_CK_KMR2
- removed U1: W25Q32JVSS, Package_SO:SOIC-8_5.23x5.23mm_P1.27mm
- added L1: L_Small, Inductor_SMD:L_0402_1005Metric, F.Cu at (22.5, 43.8)
- C2: value 0.1uF -> 1uF; moved to F.Cu
- J2: value Conn_ARM_JTAG_SWD_10 -> Conn_01x19_Male; footprint Connector_PinHeader_1.27mm:PinHeader_2x05_P1.27mm_Vertical_SMD -> Connector_PinHeader_2.54mm:PinHeader_1x19_P2.54mm_Vertical
- J3: value Conn_01x14_Male -> Conn_01x19_Male; footprint Connector_PinHeader_2.54mm:PinHeader_1x14_P2.54mm_Vertical -> Connector_PinHeader_2.54mm:PinHeader_1x19_P2.54mm_Vertical; moved to F.Cu
- moved J3 52.4 mm to (39.2, 75.1)
- moved J2 17.8 mm to (14.1, 29.3), turned to 0 degrees
- moved C3 14.0 mm to (29.0, 37.3), turned to 270 degrees
- moved C5 11.2 mm to (26.2, 33.3), turned to 180 degrees
- moved Y1 9.01 mm to (26.2, 36.3), turned to 90 degrees
- moved C1 8.81 mm to (20.6, 42.9), turned to 315 degrees
- moved C9 8.64 mm to (25.4, 53.3), turned to 315 degrees
- moved C8 8.12 mm to (32.5, 48.8), turned to 225 degrees
- moved J1 5.84 mm to (26.7, 70.6)
- moved C2 5.39 mm to (21.6, 41.9), turned to 315 degrees
- moved U2 5.08 mm to (26.7, 62.2)
- moved R7 3.09 mm to (23.4, 37.6), turned to 90 degrees
- moved C4 2.42 mm to (24.3, 54.5), turned to 315 degrees
- moved C7 0.71 mm to (28.2, 41.1), turned to 315 degrees
Connections:
- C1 pad 2: ~RST -> +3.3VA
- C2 pad 1: +3V3 -> GND
- C2 pad 2: GND -> +3.3VA
- J2 pad 1: +3V3 -> +BATT
- J2 pad 10: ~RST -> FM_CS
- J2 pad 2: SWDIO -> +3V3
- J2 pad 3: GND -> PC13
- J2 pad 4: SWDCLK -> PC14
- J2 pad 5: GND -> ~RST
- J2 pad 6: SWO -> PC15
- J2 pad 7: (no net) -> PA1
- J2 pad 8: (no net) -> PA2
- J2 pad 9: (no net) -> PA3
- J3 pad 1: +BATT -> GND
- J3 pad 10: PBO -> PA15
- J3 pad 11: PB1 -> SWO
- J3 pad 12: PB10 -> FM_MISO
- J3 pad 13: PB12 -> PB5
- J3 pad 14: GND -> PB6
- J3 pad 2: +3V3 -> PB13
- J3 pad 3: PC13 -> PB14
- J3 pad 4: PC14 -> PB15
- J3 pad 5: PC15 -> PA8
- J3 pad 6: PA1 -> PA9
- J3 pad 7: PA2 -> PA10
- J3 pad 8: PA3 -> SWDIO
- J3 pad 9: PA6 -> SWDCLK
- U3 pad 10: KEY -> (no net)
- U3 pad 20: BOOT1 -> PB2
- U3 pad 9: Net-(FB1-Pad2) -> +3.3VA
Routing:
- net PB10: track 0.00 -> 24.2 mm
- net PB2: track 0.00 -> 21.9 mm
- net PB1: track 0.00 -> 19.6 mm
- net PBO: track 0.00 -> 17.3 mm
- net FM_MOSI: track 0.00 -> 14.9 mm
- net USB_D-: track 0.00 -> 14.1 mm
- net USB_D+: track 0.00 -> 13.9 mm
- net PA6: track 0.00 -> 12.9 mm
- net FM_SCK: track 0.00 -> 11.6 mm
- net FM_CS: track 0.00 -> 10.4 mm
- net OSC_IN: track 0.00 -> 9.96 mm
- net PA1: track 0.00 -> 9.20 mm
- net PA3: track 0.00 -> 9.10 mm
- net PA2: track 0.00 -> 8.45 mm
- net +5V: track 0.00 -> 7.74 mm
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Other:
- board size 27.9 x 41.9 mm -> 27.9 x 48.5 mm

Commit message: do most of the breakout
Parts:
- J2, J3: value Conn_01x19_Male -> Conn_01x20_Male; footprint Connector_PinHeader_2.54mm:PinHeader_1x19_P2.54mm_Vertical -> Connector_PinHeader_2.54mm:PinHeader_1x20_P2.54mm_Vertical; moved to B.Cu
- moved J2 15.6 mm to (13.8, 13.8), turned to 180 degrees
- moved C1 14.1 mm to (18.2, 29.1)
- moved L1 14.0 mm to (20.0, 30.0)
- moved C2 14.0 mm to (19.1, 28.1)
- moved J3 13.3 mm to (36.6, 62.0), turned to 0 degrees
- moved C9 13.0 mm to (23.9, 40.4)
- moved U3 13.0 mm to (25.2, 34.1)
- moved C3 13.0 mm to (27.5, 24.4)
- moved C5 13.0 mm to (24.7, 20.4)
- moved C7 13.0 mm to (26.7, 28.2)
- moved Y1 13.0 mm to (24.7, 23.4)
- moved C4 13.0 mm to (22.8, 41.6)
- moved C8 13.0 mm to (31.0, 35.9)
- moved J1 13.0 mm to (25.2, 57.7)
- moved R7 13.0 mm to (21.9, 24.7)
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Connections:
- J2 pad 19: +5V -> GND
- J2 pad 3: PC13 -> (no net)
- J2 pad 4: PC14 -> (no net)
- J2 pad 5: ~RST -> (no net)
- J2 pad 6: PC15 -> ~RST
- J3 pad 5: PA8 -> (no net)
- J3 pad 6: PA9 -> (no net)
- J3 pad 7: PA10 -> (no net)
- U3 pad 2: PC13 -> (no net)
- U3 pad 29: PA8 -> (no net)
- U3 pad 3: PC14 -> (no net)
- U3 pad 30: PA9 -> (no net)
- U3 pad 31: PA10 -> (no net)
- U3 pad 4: PC15 -> (no net)
Routing:
- net PB13: track 0.00 -> 26.2 mm, vias 0 -> 1
- net PB14: track 0.00 -> 23.4 mm, vias 0 -> 1
- net PB12: track 0.00 -> 23.4 mm
- net PB15: track 0.00 -> 21.1 mm, vias 0 -> 1
- net +BATT: track 0.00 -> 20.5 mm, vias 0 -> 1
- net GND: track 3.84 -> 24.1 mm, vias 0 -> 3
- net PB9: track 0.00 -> 15.7 mm
- net USB_D-: track 14.1 -> 0.00 mm
- net USB_D+: track 13.9 -> 0.00 mm
- net PB8: track 0.00 -> 13.7 mm
- net BOOT0: track 0.00 -> 12.5 mm
- net SWDIO: track 0.00 -> 12.3 mm
- net SWDCLK: track 0.00 -> 12.2 mm
- net PA15: track 0.00 -> 11.7 mm
- net ~RST: track 0.00 -> 11.7 mm
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- added copper zone on In2.Cu, net +3V3
- added copper zone on B.Cu, net GND
- added copper zone on F.Cu, net GND
- added copper zone on In1.Cu, net GND
Other:
- board size 27.9 x 48.5 mm -> 26.4 x 51.8 mm
- copper layers 2 -> 4
