File: STM32F411CE/STM32F411CE/STM32F411CE.kicad_pcb (KiCad board)
At the start: 4 copper layers, 26.4 x 51.8 mm, 16 parts, among them J1 USB_B_Mini, J2 Conn_01x20_Male, J3 Conn_01x20_Male, U2 USBLC6-2SC6, U3 STM32F411CEUx, Y1 Crystal_GND24

Commit message: finish off the stm32f411ce
Parts:
- L1: value 37nF -> L_Small
- moved U2 1.33 mm to (25.2, 49.3)
Connections:
- net PA0 renamed KEY
- net PA4 renamed FM_CS
- net PA5 renamed FM_SCK
- net PA7 renamed FM_MOSI
- net PB4 renamed FM_MISO
- J2 pad 19: +5V -> GND
Routing:
- net +5V: track 19.6 -> 7.74 mm
- net USB_D+: track 16.4 -> 18.9 mm
- net USB_D-: track 16.5 -> 18.4 mm
- net USB_CONN_D-: track 3.78 -> 5.38 mm
- net USB_CONN_D+: track 3.78 -> 5.08 mm
Other:
- net class Default: clearance 0.1 -> 0.2
- rule trace_clearance: 0.1 -> 0.2
- rule trace_min: 0.01 -> 0.1
- rule via_min_size: 0.01 -> 0.2
- board text removed: "3.3V"
- board text removed: "5V"
- board text removed: "BAT"
- board text removed: "BOOT0"
- board text removed: "GND"
- board text removed: "NC"
- board text removed: "PA0"
- board text removed: "PA1"
- board text removed: "PA15"
- board text removed: "PA2"
- board text removed: "PA3"
- board text removed: "PA4"
- board text removed: "PA5"
- board text removed: "PA6"
- board text removed: "PA7"
- board text removed: "PB0"
- board text removed: "PB1"
- board text removed: "PB10"
- board text removed: "PB12"
- board text removed: "PB13"
- board text removed: "PB14"
- board text removed: "PB15"
- board text removed: "PB2"
- board text removed: "PB4"
- board text removed: "PB5"
- board text removed: "PB6"
- board text removed: "PB7"
- board text removed: "PB8"
- board text removed: "PB9"
- board text removed: "SWDCLK"
- board text removed: "SWDIO"
- board text removed: "SWO"
- board text removed: "~RST"
