File: STM32F411CE/STM32F411CE/STM32F411CE.sch (KiCad schematic (older format))
At the start: 28 parts, among them J1 USB_B_Mini, J2 Conn_ARM_JTAG_SWD_10, J3 Conn_01x14_Male, J4 Connector_PinHeader_2.54mm:Pi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, SW1 SW_SPDT, SW2 SW_SPST, SW3 SW_SPST, U1 W25Q32JVSS, U2 USBLC6-2SC6, U3 STM32F411CEUx, Y1 Crystal_GND24

Commit message: WIP
Parts:
- removed C6: 0.1uF, Capacitor_SMD:C_0402_1005Metric_Pad0.74x0.62mm_HandSolder, symbol Device:C
- removed FB1: 10uH, Inductor_SMD:L_0603_1608Metric, symbol Device:Ferrite_Bead
- removed J2: Conn_ARM_JTAG_SWD_10, Connector_PinHeader_1.27mm:PinHeader_2x05_P1.27mm_Vertical_SMD, symbol Connector:Conn_ARM_JTAG_SWD_10
- removed J3: Conn_01x14_Male, Connector_PinHeader_2.54mm:PinHeader_1x14_P2.54mm_Vertical, symbol Connector:Conn_01x14_Male
- removed J4: Connector_PinHeader_2.54mm:PinHeader_1x14_P2.54mm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, Connector_PinHeader_2.54mm:PinHeader_1x14_P2.54mm_Vertical, symbol Connector:Conn_01x14_Male
- removed R1, R2, R3, R4, R5, R6: 10k, Resistor_SMD:R_0402_1005Metric, symbol Device:R_US
- removed SW1: SW_SPDT, Button_Switch_SMD:SW_SPDT_PCM12, symbol Switch:SW_SPDT
- removed SW2, SW3: SW_SPST, Button_Switch_SMD:SW_Push_1P1T_NO_CK_KMR2, symbol Switch:SW_SPST
- removed U1: W25Q32JVSS, Package_SO:SOIC-8_5.23x5.23mm_P1.27mm, symbol Memory_Flash:W25Q32JVSS
- added J2, J3: Conn_01x19_Male, Connector_PinHeader_2.54mm:PinHeader_1x19_P2.54mm_Vertical, symbol Connector:Conn_01x19_Male
- added L1: L_Small, Inductor_SMD:L_0402_1005Metric, symbol Device:L_Small
- C2: value 0.1uF -> 1uF
Connections:
- net +3V3: now also J2.2 (Pin_2), L1.1; no longer C2.1
- net +5V: now also J2.19 (Pin_19)
- net +BATT: now also J2.1 (Pin_1)
- net BOOT0: now also J3.16 (Pin_16)
- net FM_CS: now also J2.10 (Pin_10)
- net FM_MISO: now also J3.12 (Pin_12)
- net FM_MOSI: now also J2.13 (Pin_13)
- net FM_SCK: now also J2.11 (Pin_11)
- net GND: now also C2.1, J3.1 (Pin_1), J3.19 (Pin_19); no longer C2.2
- net PA1: now also J2.7 (Pin_7)
- net PA10: now also J3.7 (Pin_7)
- net PA15: now also J3.10 (Pin_10)
- net PA2: now also J2.8 (Pin_8)
- net PA3: now also J2.9 (Pin_9)
- net PA6: now also J2.12 (Pin_12)
- net PA8: now also J3.5 (Pin_5)
- net PA9: now also J3.6 (Pin_6)
- net PB1: now also J2.15 (Pin_15)
- net PB10: now also J2.17 (Pin_17)
- net PB12: now also J2.18 (Pin_18)
- net PB13: now also J3.2 (Pin_2)
- net PB14: now also J3.3 (Pin_3)
- net PB15: now also J3.4 (Pin_4)
- net PB5: now also J3.13 (Pin_13)
- net PB6: now also J3.14 (Pin_14)
- net PB7: now also J3.15 (Pin_15)
- net PB8: now also J3.17 (Pin_17)
- net PB9: now also J3.18 (Pin_18)
- net PBO: now also J2.14 (Pin_14)
- net PC13: now also J2.3 (Pin_3)
- net PC14: now also J2.4 (Pin_4)
- net PC15: now also J2.6 (Pin_6)
- net SWDCLK: now also J3.9 (Pin_9)
- net SWDIO: now also J3.8 (Pin_8)
- net SWO: now also J3.11 (Pin_11)
- net ~RST: now also J2.5 (Pin_5); no longer C1.2
- net +3.3VA: now reaches U3.9 (VDDA)
- net +3.3VA: now also C1.2, C2.2, L1.2
- net BOOT1 renamed PB2
- net PB2: now also J2.16 (Pin_16)
- no-connect marks 4 -> 2
Other:
- note removed: "DEBUG / MICRO INIT"
- note removed: "FLASH"

Commit message: do most of the breakout
Parts:
- removed J2, J3: Conn_01x19_Male, Connector_PinHeader_2.54mm:PinHeader_1x19_P2.54mm_Vertical, symbol Connector:Conn_01x19_Male
- added J2, J3: Conn_01x20_Male, Connector_PinHeader_2.54mm:PinHeader_1x20_P2.54mm_Vertical, symbol Connector:Conn_01x20_Male
Connections:
- net +3V3: now also J2.2 (Pin_2)
- net +BATT: now also J2.1 (Pin_1)
- net BOOT0: now also J3.16 (Pin_16)
- net FM_CS: now also J2.10 (Pin_10)
- net FM_MISO: now also J3.12 (Pin_12)
- net FM_MOSI: now also J2.13 (Pin_13)
- net FM_SCK: now also J2.11 (Pin_11)
- net GND: now also J2.19 (Pin_19), J2.20 (Pin_20), J3.1 (Pin_1), J3.19 (Pin_19), J3.20 (Pin_20)
- net PA1: now also J2.7 (Pin_7)
- net PA15: now also J3.10 (Pin_10)
- net PA2: now also J2.8 (Pin_8)
- net PA3: now also J2.9 (Pin_9)
- net PA6: now also J2.12 (Pin_12)
- net PB1: now also J2.15 (Pin_15)
- net PB10: now also J2.17 (Pin_17)
- net PB12: now also J2.18 (Pin_18)
- net PB13: now also J3.2 (Pin_2)
- net PB14: now also J3.3 (Pin_3)
- net PB15: now also J3.4 (Pin_4)
- net PB2: now also J2.16 (Pin_16)
- net PB5: now also J3.13 (Pin_13)
- net PB6: now also J3.14 (Pin_14)
- net PB7: now also J3.15 (Pin_15)
- net PB8: now also J3.17 (Pin_17)
- net PB9: now also J3.18 (Pin_18)
- net PBO: now also J2.14 (Pin_14)
- net SWDCLK: now also J3.9 (Pin_9)
- net SWDIO: now also J3.8 (Pin_8)
- net SWO: now also J3.11 (Pin_11)
- net ~RST: now also J2.6 (Pin_6)
- net PA8: no longer names the net of U3.29 (PA8)
- net PA9: no longer names the net of U3.30 (PA9)
- no-connect marks 2 -> 10
Changed lines of the file:
@@
 L power:+3V3 #PWR0120
 U 1 1 6075BC4E
-P 9800 1450
-F 0 "#PWR0120" H 9800 1300 50  0001 C CNN
-F 1 "+3V3" H 9815 1623 50  0000 C CNN
-F 2 "" H 9800 1450 50  0001 C CNN
-F 3 "" H 9800 1450 50  0001 C CNN
-	1    9800 1450
+P 10000 1450
+F 0 "#PWR0120" H 10000 1300 50  0001 C CNN
+F 1 "+3V3" H 10015 1623 50  0000 C CNN
+F 2 "" H 10000 1450 50  0001 C CNN
+F 3 "" H 10000 1450 50  0001 C CNN
+	1    10000 1450
 	1    0    0    -1
 $EndComp
@@
 L power:GND #PWR0121
 U 1 1 6075C82A
-P 9800 1950
-F 0 "#PWR0121" H 9800 1700 50  0001 C CNN
-F 1 "GND" H 9805 1777 50  0000 C CNN
-F 2 "" H 9800 1950 50  0001 C CNN
-F 3 "" H 9800 1950 50  0001 C CNN
-	1    9800 1950
-	1    0    0    -1
-$EndComp
-Wire Wire Line
-	9800 1950 10000 1950
+P 10000 1950
+F 0 "#PWR0121" H 10000 1700 50  0001 C CNN
+F 1 "GND" H 10005 1777 50  0000 C CNN
+F 2 "" H 10000 1950 50  0001 C CNN
+F 3 "" H 10000 1950 50  0001 C CNN
+	1    10000 1950
+	1    0    0    -1
+$EndComp
 Wire Wire Line
 	10450 1950 10450 1850
@@
 	9550 1850 9550 1950
 Wire Wire Line
-	9550 1950 9800 1950
-Connection ~ 9800 1950
+	9550 1950 10000 1950
 Wire Wire Line
 	10450 1450 10450 1550
-Connection ~ 9800 1450
-Wire Wire Line
-	9800 1450 10000 1450
+Connection ~ 10000 1450
 Wire Wire Line
 	9550 1450 9550 1550
 Wire Wire Line
-	9550 1450 9800 1450
+	9550 1450 10000 1450
 Wire Wire Line
 	10000 1450 10000 1550
-Connection ~ 10000 1450
 Wire Wire Line
 	10000 1450 10450 1450
@@
 Wire Wire Line
 	9050 4250 9100 4250
-Text GLabel 2400 3850 2    50   Input ~ 0
-PC13
-Text GLabel 2400 3950 2    50   Input ~ 0
-PC14
-Text GLabel 2400 4150 2    50   Input ~ 0
-PC15
-Wire Wire Line
-	2350 3850 2400 3850
-Wire Wire Line
-	2350 3950 2400 3950
-Wire Wire Line
-	2350 4050 2400 4050
 Text GLabel 10500 4450 2    50   Input ~ 0
 PA1
@@
 Text GLabel 10500 4950 2    50   Input ~ 0
 PA6
-Text GLabel 10500 5150 2    50   Input ~ 0
-PA8
-Text GLabel 10500 5250 2    50   Input ~ 0
-PA9
 Text GLabel 10500 5350 2    50   Input ~ 0
 PA10
 Wire Wire Line
 	10400 4950 10500 4950
-Wire Wire Line
-	10400 5150 10500 5150
-Wire Wire Line
-	10400 5250 10500 5250
 Wire Wire Line
 	10500 5350 10400 5350
@@
 Wire Wire Line
 	3150 3950 3200 3950
-Wire Wire Line
-	3150 4050 3200 4050
-Wire Wire Line
-	3150 4150 3200 4150
-Wire Wire Line
-	3150 4250 3200 4250
 Text GLabel 10500 5850 2    50   Input ~ 0
 PA15
@@
 $EndComp
 Wire Wire Line
-	2550 5450 2550 5500
+	2550 5550 2550 5600
 $Comp
 L Device:Crystal_GND24 Y1
@@
 Text GLabel 10500 4750 2    50   Input ~ 0
 FM_CS
-Text GLabel 3200 4050 2    50   Input ~ 0
-PA8
-Text GLabel 3200 4150 2    50   Input ~ 0
-PA9
-Text GLabel 3200 4250 2    50   Input ~ 0
-PA10
 Wire Wire Line
 	2350 4850 2400 4850
@@
 Wire Wire Line
 	2350 5250 2400 5250
-Text GLabel 2400 4050 2    50   Input ~ 0
+Text GLabel 2400 4150 2    50   Input ~ 0
 ~RST
 Wire Wire Line
@@
 Wire Wire Line
 	3150 4750 3200 4750
-$Comp
-L Connector:Conn_01x19_Male J2
-U 1 1 60861052
+Text GLabel 2400 5350 2    50   Input ~ 0
+PB12
+Wire Wire Line
+	2350 5550 2550 5550
+$Comp
+L power:GND #PWR0109
+U 1 1 6089F64A
+P 2700 5500
+F 0 "#PWR0109" H 2700 5250 50  0001 C CNN
+F 1 "GND" H 2705 5327 50  0000 C CNN
+F 2 "" H 2700 5500 50  0001 C CNN
+F 3 "" H 2700 5500 50  0001 C CNN
+	1    2700 5500
+	1    0    0    -1
+$EndComp
+Wire Wire Line
+	2700 5450 2700 5500
+Wire Wire Line
+	3150 3650 3300 3650
+Wire Wire Line
+	3300 3600 3300 3650
+$Comp
+L Connector:Conn_01x20_Male J2
+U 1 1 608FB9C8
 P 2150 4550
 F 0 "J2" H 2258 5631 50  0000 C CNN
-F 1 "Conn_01x19_Male" H 2258 5540 50  0000 C CNN
-F 2 "Connector_PinHeader_2.54mm:PinHeader_1x19_P2.54mm_Vertical" H 2150 4550 50  0001 C CNN
+F 1 "Conn_01x20_Male" H 2258 5540 50  0000 C CNN
+F 2 "Connector_PinHeader_2.54mm:PinHeader_1x20_P2.54mm_Vertical" H 2150 4550 50  0001 C CNN
 F 3 "~" H 2150 4550 50  0001 C CNN
 	1    2150 4550
@@
 $EndComp
 $Comp
-L Connector:Conn_01x19_Male J3
-U 1 1 6086313D
+L Connector:Conn_01x20_Male J3
+U 1 1 6090F942
 P 2950 4550
 F 0 "J3" H 3058 5631 50  0000 C CNN
-F 1 "Conn_01x19_Male" H 3058 5540 50  0000 C CNN
-F 2 "Connector_PinHeader_2.54mm:PinHeader_1x19_P2.54mm_Vertical" H 2950 4550 50  0001 C CNN
+F 1 "Conn_01x20_Male" H 3058 5540 50  0000 C CNN
+F 2 "Connector_PinHeader_2.54mm:PinHeader_1x20_P2.54mm_Vertical" H 2950 4550 50  0001 C CNN
 F 3 "~" H 2950 4550 50  0001 C CNN
 	1    2950 4550
 	1    0    0    -1
 $EndComp
-Text GLabel 2400 5350 2    50   Input ~ 0
-PB12
-Wire Wire Line
-	2350 5450 2550 5450
-$Comp
-L power:GND #PWR0109
-U 1 1 6089F64A
-P 3350 5500
-F 0 "#PWR0109" H 3350 5250 50  0001 C CNN
-F 1 "GND" H 3355 5327 50  0000 C CNN
-F 2 "" H 3350 5500 50  0001 C CNN
-F 3 "" H 3350 5500 50  0001 C CNN
-	1    3350 5500
-	1    0    0    -1
-$EndComp
-Wire Wire Line
-	3350 5450 3350 5500
-Wire Wire Line
-	3150 5450 3350 5450
-Wire Wire Line
-	3150 3650 3300 3650
-Wire Wire Line
-	3300 3600 3300 3650
-$Comp
-L power:+5V #PWR?
-U 1 1 608D9D50
-P 2550 5500
-F 0 "#PWR?" H 2550 5350 50  0001 C CNN
-F 1 "+5V" H 2565 5673 50  0000 C CNN
-F 2 "" H 2550 5500 50  0001 C CNN
-F 3 "" H 2550 5500 50  0001 C CNN
-	1    2550 5500
-	-1   0    0    1
-$EndComp
+Wire Wire Line
+	2350 5450 2700 5450
+$Comp
+L power:GND #PWR0111
+U 1 1 6092DBE4
+P 3500 5500
+F 0 "#PWR0111" H 3500 5250 50  0001 C CNN
+F 1 "GND" H 3505 5327 50  0000 C CNN
+F 2 "" H 3500 5500 50  0001 C CNN
+F 3 "" H 3500 5500 50  0001 C CNN
+	1    3500 5500
+	1    0    0    -1
+$EndComp
+Wire Wire Line
+	3500 5450 3500 5500
+Wire Wire Line
+	3150 5450 3500 5450
+$Comp
+L power:GND #PWR0112
+U 1 1 609379B2
+P 3350 5600
+F 0 "#PWR0112" H 3350 5350 50  0001 C CNN
+F 1 "GND" H 3355 5427 50  0000 C CNN
+F 2 "" H 3350 5600 50  0001 C CNN
+F 3 "" H 3350 5600 50  0001 C CNN
+	1    3350 5600
+	1    0    0    -1
+$EndComp
+Wire Wire Line
+	3150 5550 3350 5550
+Wire Wire Line
+	3350 5550 3350 5600
+NoConn ~ 3150 4050
+NoConn ~ 3150 4150
+NoConn ~ 10400 5150
+NoConn ~ 10400 5250
+$Comp
+L power:GND #PWR0110
+U 1 1 609A40FC
+P 2550 5600
+F 0 "#PWR0110" H 2550 5350 50  0001 C CNN
+F 1 "GND" H 2555 5427 50  0000 C CNN
+F 2 "" H 2550 5600 50  0001 C CNN
+F 3 "" H 2550 5600 50  0001 C CNN
+	1    2550 5600
+	1    0    0    -1
+$EndComp
+NoConn ~ 2350 3850
+NoConn ~ 2350 3950
+NoConn ~ 2350 4050
+NoConn ~ 3150 4250
 $EndSCHEMATC
