File: STM32F411CE/STM32F411CE.sch (KiCad schematic (older format))
At the start: 16 parts, among them J1 USB_B_Mini, J2 Conn_01x20_Male, J3 Conn_01x20_Male, U2 USBLC6-2SC6, U3 STM32F411CEUx, Y1 Crystal_GND24

Commit message: finish STM kicad
Connections:
- net +3V3: now also J2.4 (Pin_4); no longer J2.2 (Pin_2)
- net KEY: now also J2.6 (Pin_6)
- net ~RST: now also J2.5 (Pin_5); no longer J2.6 (Pin_6)
- net PA10: no longer names the net of U3.31 (PA10)
- net PC13: no longer names the net of U3.2 (PC13)
- net PC14: no longer names the net of U3.3 (PC14)
- net PC15: no longer names the net of U3.4 (PC15)
- no-connect marks 10 -> 13
Other:
- moved on the sheet: C7, C8, C9
Changed lines of the file:
@@
 L Device:C C7
 U 1 1 6075AA39
-P 9550 1700
-F 0 "C7" H 9665 1746 50  0000 L CNN
-F 1 "0.1uF" H 9665 1655 50  0000 L CNN
-F 2 "Capacitor_SMD:C_0402_1005Metric_Pad0.74x0.62mm_HandSolder" H 9588 1550 50  0001 C CNN
-F 3 "~" H 9550 1700 50  0001 C CNN
-	1    9550 1700
+P 9350 1800
+F 0 "C7" H 9465 1846 50  0000 L CNN
+F 1 "0.1uF" H 9465 1755 50  0000 L CNN
+F 2 "Capacitor_SMD:C_0402_1005Metric_Pad0.74x0.62mm_HandSolder" H 9388 1650 50  0001 C CNN
+F 3 "~" H 9350 1800 50  0001 C CNN
+	1    9350 1800
 	1    0    0    -1
 $EndComp
@@
 L Device:C C8
 U 1 1 6075B02C
-P 10000 1700
-F 0 "C8" H 10115 1746 50  0000 L CNN
-F 1 "0.1uF" H 10115 1655 50  0000 L CNN
-F 2 "Capacitor_SMD:C_0402_1005Metric_Pad0.74x0.62mm_HandSolder" H 10038 1550 50  0001 C CNN
-F 3 "~" H 10000 1700 50  0001 C CNN
-	1    10000 1700
+P 9800 1800
+F 0 "C8" H 9915 1846 50  0000 L CNN
+F 1 "0.1uF" H 9915 1755 50  0000 L CNN
+F 2 "Capacitor_SMD:C_0402_1005Metric_Pad0.74x0.62mm_HandSolder" H 9838 1650 50  0001 C CNN
+F 3 "~" H 9800 1800 50  0001 C CNN
+	1    9800 1800
 	1    0    0    -1
 $EndComp
@@
 L Device:C C9
 U 1 1 6075B612
-P 10450 1700
-F 0 "C9" H 10565 1746 50  0000 L CNN
-F 1 "0.1uF" H 10565 1655 50  0000 L CNN
-F 2 "Capacitor_SMD:C_0402_1005Metric_Pad0.74x0.62mm_HandSolder" H 10488 1550 50  0001 C CNN
-F 3 "~" H 10450 1700 50  0001 C CNN
-	1    10450 1700
+P 10250 1800
+F 0 "C9" H 10365 1846 50  0000 L CNN
+F 1 "0.1uF" H 10365 1755 50  0000 L CNN
+F 2 "Capacitor_SMD:C_0402_1005Metric_Pad0.74x0.62mm_HandSolder" H 10288 1650 50  0001 C CNN
+F 3 "~" H 10250 1800 50  0001 C CNN
+	1    10250 1800
 	1    0    0    -1
 $EndComp
@@
 L power:+3V3 #PWR0120
 U 1 1 6075BC4E
-P 10000 1450
-F 0 "#PWR0120" H 10000 1300 50  0001 C CNN
-F 1 "+3V3" H 10015 1623 50  0000 C CNN
-F 2 "" H 10000 1450 50  0001 C CNN
-F 3 "" H 10000 1450 50  0001 C CNN
-	1    10000 1450
+P 9800 1550
+F 0 "#PWR0120" H 9800 1400 50  0001 C CNN
+F 1 "+3V3" H 9815 1723 50  0000 C CNN
+F 2 "" H 9800 1550 50  0001 C CNN
+F 3 "" H 9800 1550 50  0001 C CNN
+	1    9800 1550
 	1    0    0    -1
 $EndComp
@@
 L power:GND #PWR0121
 U 1 1 6075C82A
-P 9800 1950
-F 0 "#PWR0121" H 9800 1700 50  0001 C CNN
-F 1 "GND" H 9805 1777 50  0000 C CNN
-F 2 "" H 9800 1950 50  0001 C CNN
-F 3 "" H 9800 1950 50  0001 C CNN
-	1    9800 1950
-	1    0    0    -1
-$EndComp
-Wire Wire Line
-	9800 1950 10000 1950
-Wire Wire Line
-	10450 1950 10450 1850
-Wire Wire Line
-	10000 1850 10000 1950
-Connection ~ 10000 1950
-Wire Wire Line
-	10000 1950 10450 1950
-Wire Wire Line
-	9550 1850 9550 1950
-Wire Wire Line
-	9550 1950 9800 1950
-Connection ~ 9800 1950
-Wire Wire Line
-	10450 1450 10450 1550
-Connection ~ 10000 1450
-Wire Wire Line
-	9550 1450 9550 1550
-Wire Wire Line
-	9550 1450 10000 1450
-Wire Wire Line
-	10000 1450 10000 1550
-Wire Wire Line
-	10000 1450 10450 1450
+P 9800 2050
+F 0 "#PWR0121" H 9800 1800 50  0001 C CNN
+F 1 "GND" H 9805 1877 50  0000 C CNN
+F 2 "" H 9800 2050 50  0001 C CNN
+F 3 "" H 9800 2050 50  0001 C CNN
+	1    9800 2050
+	1    0    0    -1
+$EndComp
+Wire Wire Line
+	10250 2050 10250 1950
+Wire Wire Line
+	9800 1950 9800 2050
+Connection ~ 9800 2050
+Wire Wire Line
+	9800 2050 10250 2050
+Wire Wire Line
+	9350 1950 9350 2050
+Wire Wire Line
+	9350 2050 9800 2050
+Wire Wire Line
+	10250 1550 10250 1650
+Connection ~ 9800 1550
+Wire Wire Line
+	9350 1550 9350 1650
+Wire Wire Line
+	9350 1550 9800 1550
+Wire Wire Line
+	9800 1550 9800 1650
+Wire Wire Line
+	9800 1550 10250 1550
 $Comp
 L Device:C C4
@@
 Wire Wire Line
 	2450 3650 2450 3600
-Text GLabel 9050 4050 0    50   Input ~ 0
-PC13
-Text GLabel 9050 4150 0    50   Input ~ 0
-PC14
-Text GLabel 9050 4250 0    50   Input ~ 0
-PC15
-Wire Wire Line
-	9050 4050 9100 4050
-Wire Wire Line
-	9050 4150 9100 4150
-Wire Wire Line
-	9050 4250 9100 4250
 Text GLabel 10500 4450 2    50   Input ~ 0
 PA1
@@
 Text GLabel 10500 4950 2    50   Input ~ 0
 PA6
-Text GLabel 10500 5350 2    50   Input ~ 0
-PA10
 Wire Wire Line
 	10400 4950 10500 4950
-Wire Wire Line
-	10500 5350 10400 5350
 Text GLabel 2400 4750 2    50   Input ~ 0
 PA6
@@
 L power:+3V3 #PWR0127
 U 1 1 6083F32C
-P 2700 3600
-F 0 "#PWR0127" H 2700 3450 50  0001 C CNN
-F 1 "+3V3" H 2715 3773 50  0000 C CNN
-F 2 "" H 2700 3600 50  0001 C CNN
-F 3 "" H 2700 3600 50  0001 C CNN
-	1    2700 3600
-	1    0    0    -1
-$EndComp
-Wire Wire Line
-	2350 3750 2700 3750
-Wire Wire Line
-	2700 3750 2700 3600
+P 2700 3800
+F 0 "#PWR0127" H 2700 3650 50  0001 C CNN
+F 1 "+3V3" H 2715 3973 50  0000 C CNN
+F 2 "" H 2700 3800 50  0001 C CNN
+F 3 "" H 2700 3800 50  0001 C CNN
+	1    2700 3800
+	1    0    0    -1
+$EndComp
+Wire Wire Line
+	2350 3950 2700 3950
+Wire Wire Line
+	2700 3950 2700 3800
 Wire Wire Line
 	3150 4350 3200 4350
@@
 Wire Wire Line
 	2350 5250 2400 5250
-Text GLabel 2400 4150 2    50   Input ~ 0
+Text GLabel 2400 4050 2    50   Input ~ 0
 ~RST
 Wire Wire Line
@@
 	1    0    0    -1
 $EndComp
+NoConn ~ 2350 3750
 NoConn ~ 2350 3850
-NoConn ~ 2350 3950
-NoConn ~ 2350 4050
 NoConn ~ 3150 4250
+NoConn ~ 10400 5350
+Wire Wire Line
+	2350 4050 2400 4050
+Text GLabel 2400 4150 2    50   Input ~ 0
+KEY
+NoConn ~ 9100 4050
+NoConn ~ 9100 4150
+NoConn ~ 9100 4250
 $EndSCHEMATC

Commit message: finish off the stm32f411ce
Parts:
- L1: value L_Small -> 37nF
Connections:
- net +5V: now also J2.19 (Pin_19)
- net GND: no longer J2.19 (Pin_19)
- net FM_CS renamed PA4
- net FM_MISO renamed PB4
- net FM_MOSI renamed PA7
- net FM_SCK renamed PA5
- net KEY renamed PA0
Other:
- note added: "BYPASS CAPS"
- note added: "HEADERS"
- note added: "HSE"
- note added: "LC FILTER FOR ADC"
- moved on the sheet: C1, C2, C3, C4, C5, C7, C8, C9, J2, J3, L1, R7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
